File: pcb/stm32f765-breakout-board/connectors.kicad_sch (KiCad schematic)
At the start: 9 parts, among them J3 SWD, J4 Conn_01x05, J5 Conn_01x04, J6 Conn_01x12, J7 Conn_01x12, J8 Conn_01x03, J9 Conn_I2C2

Commit message: added lsm6dsl to pcb and ordered v3
Parts:
- R6, R7: value 1k5 -> 10k; Robu SKU R143534 -> R242850
Changed lines of the file:
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@@
 			)
 		)
-		(property "Value" "1k5"
+		(property "Value" "10k"
 			(at 124.968 38.1 90)
 			(effects
@@
 			)
 		)
-		(property "Robu SKU" "R143534"
+		(property "Robu SKU" "R242850"
 			(at 123.19 38.1 90)
 			(effects
@@
 			)
 		)
-		(property "Value" "1k5"
+		(property "Value" "10k"
 			(at 130.048 40.64 90)
 			(effects
@@
 			)
 		)
-		(property "Robu SKU" "R143534"
+		(property "Robu SKU" "R242850"
 			(at 128.27 40.64 90)
 			(effects

Commit message: Updated titleblock on f765 breakout pcb
Other:
- company: (none) -> Pranav Chandra N. V.
- title: (none) -> STM32F765VIT6 Breakout Board
Changed lines of the file:
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@@
 	(generator_version "9.0")
 	(paper "A4")
+	(title_block
+		(title "STM32F765VIT6 Breakout Board")
+		(date "2026-04-17")
+		(rev "v5")
+		(company "Pranav Chandra N. V.")
+		(comment 1 "v2: Added GPIO headers for various communication ports")
+		(comment 2 "v3: Changed headers to just be general GPIO ports on four sides.")
+	)
 	(text "I2C2 Connector"
 		(exclude_from_sim no)
