File: pcb/stm32f765-breakout-board/usb_connector.kicad_sch (KiCad schematic)
At the start: 4 parts, among them J1 16P_USB_C, U3 USBLC6-2SC6

Commit message: Updated titleblock on f765 breakout pcb
Other:
- company: (none) -> Pranav Chandra N. V.
- title: (none) -> STM32F765VIT6 Breakout Board
Changed lines of the file:
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@@
 	(generator_version "9.0")
 	(paper "A4")
+	(title_block
+		(title "STM32F765VIT6 Breakout Board")
+		(date "2026-04-17")
+		(rev "v5")
+		(company "Pranav Chandra N. V.")
+		(comment 1 "v3: Added ESD Protection and Config Resistors for USB C")
+	)
 	(text "USB-C Receptacle\n"
 		(exclude_from_sim no)
