File: pcb/kamikaze-drone/peripherals.kicad_sch (KiCad schematic)
At the start: 20 parts, among them J4 Conn_02x09_Odd_Even, U5 LSM6DSL, U6 W25Q64JVSS, U7 BMP280, U8 VL53L1CXV0FY1

Commit message: feat: added touch points to PCB
Took advice from reddit to improve the PCB schematic
Parts:
- added TP3, TP4: TestPoint, TestPoint:TestPoint_Pad_D1.0mm, symbol Connector:TestPoint
Connections:
- net I2C1_SCL: now also TP4.1
- net I2C1_SDA: now also TP3.1
Changed lines of the file:
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@@
 	)
 	(junction
+		(at 71.12 125.73)
+		(diameter 0)
+		(color 0 0 0 0)
+	)
+	(junction
 		(at 123.19 177.8)
 		(diameter 0)
@@
 		(color 0 0 0 0)
 	)
+	(junction
+		(at 66.04 123.19)
+		(diameter 0)
+		(color 0 0 0 0)
+	)
 	(no_connect
 		(at 63.5 160.02)
@@
 	(wire
 		(pts
-			(xy 36.83 123.19) (xy 72.39 123.19)
+			(xy 36.83 123.19) (xy 66.04 123.19)
 		)
 		(stroke
@@
 	(wire
 		(pts
+			(xy 71.12 114.3) (xy 71.12 125.73)
+		)
+		(stroke
+			(width 0)
+			(type default)
+		)
+	)
+	(wire
+		(pts
 			(xy 127 91.44) (xy 127 93.98)
 		)
@@
 	(wire
 		(pts
+			(xy 66.04 123.19) (xy 72.39 123.19)
+		)
+		(stroke
+			(width 0)
+			(type default)
+		)
+	)
+	(wire
+		(pts
 			(xy 149.86 168.91) (xy 149.86 171.45)
 		)
@@
 	(wire
 		(pts
-			(xy 43.18 125.73) (xy 72.39 125.73)
+			(xy 66.04 114.3) (xy 66.04 123.19)
+		)
+		(stroke
+			(width 0)
+			(type default)
+		)
+	)
+	(wire
+		(pts
+			(xy 43.18 125.73) (xy 71.12 125.73)
 		)
 		(stroke
@@
 	(wire
 		(pts
+			(xy 71.12 125.73) (xy 72.39 125.73)
+		)
+		(stroke
+			(width 0)
+			(type default)
+		)
+	)
+	(wire
+		(pts
 			(xy 123.19 156.21) (xy 123.19 157.48)
 		)
@@
 	)
 	(symbol
+		(lib_id "Connector:TestPoint")
+		(at 71.12 114.3 0)
+		(unit 1)
+		(exclude_from_sim no)
+		(in_bom yes)
+		(on_board yes)
+		(dnp no)
+		(property "Reference" "TP4"
+			(at 69.85 109.22 0)
+			(effects
+				(font
+					(size 1.27 1.27)
+				)
+				(justify left)
+			)
+		)
+		(property "Value" "TestPoint"
+			(at 73.66 112.2679 0)
+			(effects
+				(font
+					(size 1.27 1.27)
+				)
+				(justify left)
+				(hide yes)
+			)
+		)
+		(property "Footprint" "TestPoint:TestPoint_Pad_D1.0mm"
+			(at 76.2 114.3 0)
+			(effects
+				(font
+					(size 1.27 1.27)
+				)
+				(hide yes)
+			)
+		)
+		(property "Datasheet" "~"
+			(at 76.2 114.3 0)
+			(effects
+				(font
+					(size 1.27 1.27)
+				)
+				(hide yes)
+			)
+		)
+		(property "Description" "test point"
+			(at 71.12 114.3 0)
+			(effects
+				(font
+					(size 1.27 1.27)
+				)
+				(hide yes)
+			)
+		)
+		(pin "1"
+		)
+		(instances
+			(project "kamikaze-drone"
+				(path "/cb5e77c2-5384-4927-a501-b53a4a151a18/ee3fd35c-d83c-45a2-a285-e3082223ddcc"
+					(reference "TP4")
+					(unit 1)
+				)
+			)
+		)
+	)
+	(symbol
 		(lib_id "Device:R_Small")
 		(at 60.96 118.11 180)
@@
 					(unit 1)
 				)
+			)
+		)
+	)
+	(symbol
+		(lib_id "Connector:TestPoint")
+		(at 66.04 114.3 0)
+		(unit 1)
+		(exclude_from_sim no)
+		(in_bom yes)
+		(on_board yes)
+		(dnp no)
+		(property "Reference" "TP3"
+			(at 64.77 109.22 0)
+			(effects
+				(font
+					(size 1.27 1.27)
+				)
+				(justify left)
+			)
+		)
+		(property "Value" "TestPoint"
+			(at 68.58 112.2679 0)
+			(effects
+				(font
+					(size 1.27 1.27)
+				)
+				(justify left)
+				(hide yes)
+			)
+		)
+		(property "Footprint" "TestPoint:TestPoint_Pad_D1.0mm"
+			(at 71.12 114.3 0)
+			(effects
+				(font
+					(size 1.27 1.27)
+				)
+				(hide yes)
+			)
+		)
+		(property "Datasheet" "~"
+			(at 71.12 114.3 0)
+			(effects
+				(font
+					(size 1.27 1.27)
+				)
+				(hide yes)
+			)
+		)
+		(property "Description" "test point"
+			(at 66.04 114.3 0)
+			(effects
+				(font
+					(size 1.27 1.27)
+				)
+				(hide yes)
+			)
+		)
+		(pin "1"
+		)
+		(instances
+			(project "kamikaze-drone"
+				(path "/cb5e77c2-5384-4927-a501-b53a4a151a18/ee3fd35c-d83c-45a2-a285-e3082223ddcc"
+					(reference "TP3")
+					(unit 1)
+				)
