File: pcb/kamikaze-drone/power_management.kicad_sch (KiCad schematic)
At the start: 34 parts, among them J2 Battery Input, J3 16P_USB_C, U2 USBLC6-2P6, U3 MCP73871-2CC, U4 AMS1117-3.3

Commit message: WIP - arranging components in updated PCB
Parts:
- C13, C14, C18, C19: footprint Capacitor_SMD:C_0805_2012Metric_Pad1.18x1.45mm_HandSolder -> Capacitor_SMD:C_0603_1608Metric_Pad1.08x0.95mm_HandSolder
Changed lines of the file:
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@@
 			)
 		)
-		(property "Footprint" "Capacitor_SMD:C_0805_2012Metric_Pad1.18x1.45mm_HandSolder"
+		(property "Footprint" "Capacitor_SMD:C_0603_1608Metric_Pad1.08x0.95mm_HandSolder"
 			(at 116.84 127 0)
 			(effects
@@
 			)
 		)
-		(property "Footprint" "Capacitor_SMD:C_0805_2012Metric_Pad1.18x1.45mm_HandSolder"
+		(property "Footprint" "Capacitor_SMD:C_0603_1608Metric_Pad1.08x0.95mm_HandSolder"
 			(at 214.63 44.45 0)
 			(effects
@@
 			)
 		)
-		(property "Footprint" "Capacitor_SMD:C_0805_2012Metric_Pad1.18x1.45mm_HandSolder"
+		(property "Footprint" "Capacitor_SMD:C_0603_1608Metric_Pad1.08x0.95mm_HandSolder"
 			(at 107.95 127 0)
 			(effects
@@
 			)
 		)
-		(property "Footprint" "Capacitor_SMD:C_0805_2012Metric_Pad1.18x1.45mm_HandSolder"
+		(property "Footprint" "Capacitor_SMD:C_0603_1608Metric_Pad1.08x0.95mm_HandSolder"
 			(at 252.73 44.45 0)
 			(effects

Commit message: v2.0 of PCB completed
Updated routing to have USB port in center of top.
Shrank overall size to 50x50 mm
Layout is now ground+signal >> ground >> 3V3 >> signal

TODO: Add stitching vias between ground on top and second layer?
Other:
- note added: "MCP7871 Battery Charger + Regulator Setup"
- note added: "USB Connection Input"
Changed lines of the file:
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@@
 	(title_block
 		(title "Power Management Configuration")
-		(date "2026-05-21")
-		(rev "v1.0")
+		(date "2026-05-24")
+		(rev "v1.1")
 		(company "Pranav Chandra N. V.")
 		(comment 1 "v1.0 - First Iteration")
+		(comment 2 "v1.1 - Updated netlabels and neatened the schematic")
+	)
+	(text "MCP7871 Battery Charger + Regulator Setup"
+		(exclude_from_sim no)
+		(at 35.56 111.252 0)
+		(effects
+			(font
+				(size 1.27 1.27)
+			)
+		)
 	)
 	(text "Analog Voltage Filtering"
@@
 		(effects
 			(font
+				(size 1.27 1.27)
+			)
+		)
+	)
+	(text "USB Connection Input"
+		(exclude_from_sim no)
+		(at 24.13 50.292 0)
+		(effects
+			(font

Commit message: feat: added touch points to PCB
Took advice from reddit to improve the PCB schematic
Parts:
- added TP2, TP5: TestPoint, TestPoint:TestPoint_Pad_D1.0mm, symbol Connector:TestPoint
Connections:
- net VBAT: now also TP5.1
- net VBUS: now also TP2.1
Changed lines of the file:
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@@
 	)
 	(junction
+		(at 26.67 137.16)
+		(diameter 0)
+		(color 0 0 0 0)
+	)
+	(junction
 		(at 214.63 33.02)
 		(diameter 0)
@@
 	)
 	(junction
+		(at 74.93 144.78)
+		(diameter 0)
+		(color 0 0 0 0)
+	)
+	(junction
 		(at 52.07 25.4)
 		(diameter 0)
@@
 	(wire
 		(pts
-			(xy 27.94 134.62) (xy 27.94 137.16)
+			(xy 16.51 134.62) (xy 16.51 137.16)
 		)
 		(stroke
@@
 	(wire
 		(pts
-			(xy 69.85 144.78) (xy 85.09 144.78)
+			(xy 69.85 144.78) (xy 74.93 144.78)
 		)
 		(stroke
@@
 	(wire
 		(pts
+			(xy 26.67 137.16) (xy 34.29 137.16)
+		)
+		(stroke
+			(width 0)
+			(type default)
+		)
+	)
+	(wire
+		(pts
 			(xy 74.93 38.1) (xy 85.09 38.1)
 		)
@@
 	(wire
 		(pts
+			(xy 69.85 137.16) (xy 85.09 137.16)
+		)
+		(stroke
+			(width 0)
+			(type default)
+		)
+	)
+	(wire
+		(pts
 			(xy 264.16 53.34) (xy 264.16 49.53)
 		)
@@
 	(wire
 		(pts
+			(xy 74.93 144.78) (xy 85.09 144.78)
+		)
+		(stroke
+			(width 0)
+			(type default)
+		)
+	)
+	(wire
+		(pts
 			(xy 107.95 166.37) (xy 107.95 170.18)
 		)
@@
 	(wire
 		(pts
-			(xy 85.09 137.16) (xy 69.85 137.16)
-		)
-		(stroke
-			(width 0)
-			(type default)
-		)
-	)
-	(wire
-		(pts
 			(xy 16.51 142.24) (xy 19.05 142.24)
 		)
@@
 	(wire
 		(pts
-			(xy 27.94 137.16) (xy 34.29 137.16)
+			(xy 16.51 137.16) (xy 26.67 137.16)
 		)
 		(stroke
@@
 	)
 	(symbol
+		(lib_id "Connector:TestPoint")
+		(at 26.67 137.16 0)
+		(unit 1)
+		(exclude_from_sim no)
+		(in_bom yes)
+		(on_board yes)
+		(dnp no)
+		(property "Reference" "TP2"
+			(at 25.4 132.08 0)
+			(effects
+				(font
+					(size 1.27 1.27)
+				)
+				(justify left)
+			)
+		)
+		(property "Value" "TestPoint"
+			(at 29.21 135.1279 0)
+			(effects
+				(font
+					(size 1.27 1.27)
+				)
+				(justify left)
+				(hide yes)
+			)
+		)
+		(property "Footprint" "TestPoint:TestPoint_Pad_D1.0mm"
+			(at 31.75 137.16 0)
+			(effects
+				(font
+					(size 1.27 1.27)
+				)
+				(hide yes)
+			)
+		)
+		(property "Datasheet" "~"
+			(at 31.75 137.16 0)
+			(effects
+				(font
+					(size 1.27 1.27)
+				)
+				(hide yes)
+			)
+		)
+		(property "Description" "test point"
+			(at 26.67 137.16 0)
+			(effects
+				(font
+					(size 1.27 1.27)
+				)
+				(hide yes)
+			)
+		)
+		(pin "1"
+		)
+		(instances
+			(project "kamikaze-drone"
+				(path "/cb5e77c2-5384-4927-a501-b53a4a151a18/e1f2b4cf-2ed6-4660-b538-bb1ec10505b9"
+					(reference "TP2")
+					(unit 1)
+				)
+			)
+		)
+	)
+	(symbol
 		(lib_id "power:GND")
 		(at 52.07 180.34 0)
@@
 	(symbol
 		(lib_id "power:VBUS")
-		(at 27.94 134.62 0)
+		(at 16.51 134.62 0)
 		(unit 1)
 		(exclude_from_sim no)
@@
 		(dnp no)
 		(property "Reference" "#PWR019"
-			(at 27.94 138.43 0)
+			(at 16.51 138.43 0)
 			(effects
 				(font
@@
 		)
 		(property "Value" "VBUS"
-			(at 27.94 130.81 0)
+			(at 16.51 130.81 0)
 			(effects
 				(font
@@
 		)
 		(property "Footprint" ""
-			(at 27.94 134.62 0)
+			(at 16.51 134.62 0)
 			(effects
 				(font
@@
 		)
 		(property "Datasheet" ""
-			(at 27.94 134.62 0)
+			(at 16.51 134.62 0)
 			(effects
 				(font
@@
 		)
 		(property "Description" "Power symbol creates a global label with name \"VBUS\""
-			(at 27.94 134.62 0)
+			(at 16.51 134.62 0)
 			(effects
 				(font
@@
 					(unit 1)
 				)
+			)
+		)
+	)
+	(symbol
+		(lib_id "Connector:TestPoint")
+		(at 74.93 144.78 0)
+		(unit 1)
+		(exclude_from_sim no)
+		(in_bom yes)
+		(on_board yes)
+		(dnp no)
+		(property "Reference" "TP5"
+			(at 73.66 139.7 0)
+			(effects
+				(font
+					(size 1.27 1.27)
+				)
+				(justify left)
+			)
+		)
+		(property "Value" "TestPoint"
+			(at 77.47 142.7479 0)
+			(effects
+				(font
+					(size 1.27 1.27)
+				)
+				(justify left)
+				(hide yes)
+			)
+		)
+		(property "Footprint" "TestPoint:TestPoint_Pad_D1.0mm"
+			(at 80.01 144.78 0)
+			(effects
+				(font
+					(size 1.27 1.27)
+				)
+				(hide yes)
+			)
+		)
+		(property "Datasheet" "~"
+			(at 80.01 144.78 0)
+			(effects
+				(font
+					(size 1.27 1.27)
+				)
+				(hide yes)
+			)
+		)
+		(property "Description" "test point"
+			(at 74.93 144.78 0)
+			(effects
+				(font
+					(size 1.27 1.27)
+				)
+				(hide yes)
+			)
+		)
+		(pin "1"
+		)
+		(instances
+			(project "kamikaze-drone"
+				(path "/cb5e77c2-5384-4927-a501-b53a4a151a18/e1f2b4cf-2ed6-4660-b538-bb1ec10505b9"
+					(reference "TP5")
+					(unit 1)
+				)

Commit message: v3 of PCB made. ov7670 implementation guide added
Connections:
- net +3V3: no longer U2.5 (VBUS)
- net VBUS: now also U2.5 (VBUS)
Changed lines of the file:
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@@
 	)
 	(symbol
+		(lib_id "power:VBUS")
+		(at 45.72 67.31 0)
+		(unit 1)
+		(exclude_from_sim no)
+		(in_bom yes)
+		(on_board yes)
+		(dnp no)
+		(fields_autoplaced yes)
+		(property "Reference" "#PWR022"
+			(at 45.72 71.12 0)
+			(effects
+				(font
+					(size 1.27 1.27)
+				)
+				(hide yes)
+			)
+		)
+		(property "Value" "VBUS"
+			(at 45.72 62.23 0)
+			(effects
+				(font
+					(size 1.27 1.27)
+				)
+			)
+		)
+		(property "Footprint" ""
+			(at 45.72 67.31 0)
+			(effects
+				(font
+					(size 1.27 1.27)
+				)
+				(hide yes)
+			)
+		)
+		(property "Datasheet" ""
+			(at 45.72 67.31 0)
+			(effects
+				(font
+					(size 1.27 1.27)
+				)
+				(hide yes)
+			)
+		)
+		(property "Description" "Power symbol creates a global label with name \"VBUS\""
+			(at 45.72 67.31 0)
+			(effects
+				(font
+					(size 1.27 1.27)
+				)
+				(hide yes)
+			)
+		)
+		(pin "1"
+		)
+		(instances
+			(project "kamikaze-drone"
+				(path "/cb5e77c2-5384-4927-a501-b53a4a151a18/e1f2b4cf-2ed6-4660-b538-bb1ec10505b9"
+					(reference "#PWR022")
+					(unit 1)
+				)
+			)
+		)
+	)
+	(symbol
 		(lib_id "Device:C_Small")
 		(at 162.56 31.75 0)
@@
 					(unit 1)
 				)
-			)
-		)
-	)
-	(symbol
-		(lib_id "power:+3V3")
-		(at 45.72 67.31 0)
-		(unit 1)
-		(exclude_from_sim no)
-		(in_bom yes)
-		(on_board yes)
-		(dnp no)
-		(property "Reference" "#PWR022"
-			(at 45.72 71.12 0)
-			(effects
-				(font
-					(size 1.27 1.27)
-				)
-				(hide yes)
-			)
-		)
-		(property "Value" "+3V3"
-			(at 45.212 63.754 0)
-			(effects
-				(font
-					(size 1.27 1.27)
-				)
-			)
-		)
-		(property "Footprint" ""
-			(at 45.72 67.31 0)
-			(effects
-				(font
-					(size 1.27 1.27)
-				)
-				(hide yes)
-			)
-		)
-		(property "Datasheet" ""
-			(at 45.72 67.31 0)
-			(effects
-				(font
-					(size 1.27 1.27)
-				)
-				(hide yes)
-			)
-		)
-		(property "Description" "Power symbol creates a global label with name \"+3V3\""
-			(at 45.72 67.31 0)
-			(effects
-				(font
-					(size 1.27 1.27)
-				)
-				(hide yes)
-			)
-		)
-		(pin "1"
-		)
-		(instances
-			(project "kamikaze-drone"
-				(path "/cb5e77c2-5384-4927-a501-b53a4a151a18/e1f2b4cf-2ed6-4660-b538-bb1ec10505b9"
-					(reference "#PWR022")
-					(unit 1)
-				)
